File: oresat1-plusz-end-cap/oresat1-plusz-end-cap.kicad_pcb (KiCad board)
At the start: 4 copper layers, 105.6 x 105.6 mm, 55 parts, among them J1 M55-7011242R, J2 U.FL-R-SMA, U1 RM3100, U2 RM3100

Commit message: OreSat1 +Z End Cap updates
Fixed SDA/SCL issue, updated to v1.1.
Connections:
- U1 pad 1: /MAG-SCL -> /MAG-SDA
- U1 pad 27: /MAG-SDA -> /MAG-SCL
- U2 pad 1: /MAG-SCL -> /MAG-SDA
- U2 pad 27: /MAG-SDA -> /MAG-SCL
Routing:
- net /MAG-SCL: track 172.0 -> 172.7 mm
- net /MAG-SDA: track 170.4 -> 169.8 mm
Other:
- board text added: "1"
