File: oresat1-plusz-end-cap/oresat1-plusz-end-cap.kicad_sch (KiCad schematic)
At the start: 44 parts, among them J1 M55-7011242R, J2 U.FL-R-SMA, U1 RM3100, U2 RM3100

Commit message: OreSat1 +Z End Cap updates
Fixed SDA/SCL issue, updated to v1.1.
Connections:
- net MAG-SCL: now also U1.27 (SCLK), U2.27 (SCLK); no longer U1.1 (MOSI/SDA), U2.1 (MOSI/SDA)
- net MAG-SDA: now also U1.1 (MOSI/SDA), U2.1 (MOSI/SDA); no longer U1.27 (SCLK), U2.27 (SCLK)
Other:
- note added: "PIN 1 INDICATOR HERE"
